File: ssk-controller.kicad_pcb (KiCad board)
At the start: 2 copper layers, 285 x 95.1 mm, 205 parts, among them SW1 5.2x5.2mm, U1 ATmega32U4-MU, U2 PRTR5V0U2X, Y1 16Mhz

Commit message: Finish board
Parts:
- removed C1, C10, C11, C12, C13, C14, C15, C16, C17, C18, C19, C20, C21, C9: 0.1uF, Capacitors_SMD:C_0603
- removed D1, D10, D11, D12, D13, D14, D16, D17, D18, D19, D2, D20, D21, D22, D23, D24, D25, D26, D27, D28, D29, D3, D30, D31, D32, D33, D34, D35, D36, D37, D38, D39, D4, D40, D41, D42, D43, D44, D45, D46, D47, D48, D49, D5, D50, D51, D52, D53, D54, D55, D56, D57, D58, D59, D6, D60, D61, D62, D63, D64, D65, D67, D68, D7, D8, D9: SOD-123, Diodes_SMD:D_SOD-123
- removed the G*** at (77.8, 60.3)
- removed the G*** at (262.7, 98.4) (x2)
- removed K_#1, K_#10, K_#2, K_#3, K_#4, K_#5, K_#6, K_#7, K_#8, K_#9, K_'1, K_,1, K_-1, K_.1, K_/1, K_;1, K_=1, K_A1, K_B1, K_C1, K_D1, K_E1, K_ENTER2, K_ENTER3, K_ENTER4, K_ESC1, K_ESC2, K_F1, K_G1, K_H1, K_I1, K_J1, K_K1, K_L1, K_M1, K_N1, K_O1, K_P1, K_Q1, K_R1, K_RWIN3, K_S1, K_SBACK1, K_SBACK2, K_SHIFT3, K_SRSHIFT2, K_T1, K_U1, K_V1, K_W1, K_WIN2, K_X1, K_Y1, K_Z1, K_[1, K_\2, K_]1: MX-1U, MX_Alps_Hybrid:ALPS-1U
- removed K_ALT1, K_CAPS2, K_CTRL1, K_RALT2, K_RCTRL2, K_RMENU2, K_RWIN1, K_RWIN2, K_SHIFT2, K_SPACE5, K_WIN1, K_WIN3: MX-1.25U, MX_Alps_Hybrid:ALPS-1.25U
- removed K_ALT2, K_ALT3, K_CAPS3, K_CTRL2, K_RALT1, K_RALT3, K_RCTRL3, K_TAB1, K_\1: MX-1.5U, MX_Alps_Hybrid:ALPS-1.5U
- removed K_BACK1: MX-2U, MX_Alps_Hybrid:ALPS-2U
- removed K_CAPS1, K_SRSHIFT1: MX-1.75U, MX_Alps_Hybrid:ALPS-1.75U
- removed K_ENTER1, K_SHIFT1, K_SPACE3: MX-2.25U, MX_Alps_Hybrid:ALPS-2.25U
- removed K_RSHIFT1, K_SPACE4: MX-2.75U, MX_Alps_Hybrid:ALPS-2.75U
- removed K_SPACE1: MX-7U, MX_Alps_Hybrid:ALPS-7U
- removed K_SPACE2: MX-6.25U, MX_Alps_Hybrid:ALPS-6.25U
- removed the REF** at (165.1, 69.8)
- removed RGB1, RGB10, RGB11, RGB12, RGB13, RGB14, RGB2, RGB3, RGB4, RGB5, RGB6, RGB7, RGB8, RGB9: WS2812B, WS2812B:WS2812B
- added G***: LOGO, locallib:Quasar-Logo, F.Cu at (104.2, 95.0)
- added G***: LOGO, locallib:Quasar-Desc, F.Cu at (147.5, 95.0)
- added G***: LOGO, locallib:ai-ring-6mm-Combined, F.Cu at (234.0, 94.5)
- added G***: LOGO, locallib:ai-ring-6mm-Combined, B.Cu at (234.0, 94.5)
- added J1: Conn_01x16, Pin_Headers:Pin_Header_Straight_1x16_Pitch2.54mm, F.Cu at (144.0, 54.0)
- added J2: Conn_01x08, Pin_Headers:Pin_Header_Straight_1x08_Pitch2.54mm, F.Cu at (217.0, 57.0)
- added J3: Conn_01x01, Pin_Headers:Pin_Header_Straight_1x01_Pitch2.54mm, F.Cu at (95.0, 75.0)
- added REF**: MountingHole_3.5mm, Mounting_Holes:MountingHole_3.5mm, F.Cu at (127.0, 55.0)
- added REF**: MountingHole_3.5mm, Mounting_Holes:MountingHole_3.5mm, F.Cu at (103.0, 55.0)
- added REF**: breakaway-mousebites, random-keyboard-parts:breakaway-mousebites, F.Cu at (240.0, 75.0)
- added REF**: breakaway-mousebites, random-keyboard-parts:breakaway-mousebites, F.Cu at (240.0, 60.0)
- added REF**: breakaway-mousebites, random-keyboard-parts:breakaway-mousebites, F.Cu at (240.0, 90.0)
- C2, C3, C4, C5, C6, C7, C8: footprint Capacitors_SMD:C_0603 -> Capacitors_SMD:C_0805; moved to F.Cu
- F1, R67, R68, R70, R71, R73, R74, U2, USB1, Y1: moved to F.Cu
- SW1: value 5.2x5.2mm -> SW_Push; footprint Molex-0548190589:SKQG-1155865 -> random-keyboard-parts:SKQG-1155865; moved to F.Cu
- U1: value ATmega32U4-MU -> ATmega32U4-AU; footprint Housings_DFN_QFN:QFN-44-1EP_7x7mm_Pitch0.5mm -> Housings_QFP:TQFP-44_10x10mm_Pitch0.8mm; moved to F.Cu
- moved C7 106.0 mm to (146.5, 85.5)
- moved C8 98.5 mm to (142.0, 89.5)
- moved Y1 98.4 mm to (142.0, 85.5), turned to 180 degrees
- moved C3 96.8 mm to (147.0, 63.5), turned to 0 degrees
- moved C5 94.7 mm to (151.0, 77.5), turned to 90 degrees
- moved R73 89.3 mm to (119.0, 59.5), turned to 90 degrees
- moved U1 89.0 mm to (142.0, 72.5), turned to 0 degrees
- moved R71 88.2 mm to (151.0, 67.0), turned to 270 degrees
- moved C4 87.7 mm to (136.0, 83.5), turned to 90 degrees
- moved F1 87.4 mm to (120.0, 64.5)
- moved SW1 83.2 mm to (115.0, 75.0), turned to 180 degrees
- moved R67 81.2 mm to (116.5, 64.0)
- moved C6 79.5 mm to (132.0, 72.5), turned to 180 degrees
- moved U2 78.8 mm to (115.0, 59.5)
- moved USB1 78.7 mm to (115.0, 47.0), turned to 180 degrees
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Connections:
- U1 pad 10: ROW1 -> COL2
- U1 pad 11: ROW2 -> COL3
- U1 pad 12: Net-(U1-Pad12) -> COL4
- U1 pad 18: Net-(U1-Pad18) -> ROW0
- U1 pad 19: Net-(U1-Pad19) -> ROW1
- U1 pad 20: RGBLED -> ROW2
- U1 pad 21: COL13 -> ROW3
- U1 pad 22: COL12 -> ROW4
- U1 pad 25: COL11 -> ROW5
- U1 pad 26: COL10 -> ROW6
- U1 pad 27: COL9 -> ROW7
- U1 pad 28: COL8 -> COL15
- U1 pad 29: COL7 -> COL14
- U1 pad 30: COL6 -> COL13
- U1 pad 31: COL5 -> COL12
- U1 pad 32: COL4 -> COL11
- U1 pad 36: COL1 -> COL10
- U1 pad 37: COL3 -> COL9
- U1 pad 38: COL2 -> COL8
- U1 pad 39: COL0 -> COL7
- U1 pad 40: ROW4 -> COL6
- U1 pad 41: ROW3 -> COL5
- U1 pad 8: Net-(U1-Pad8) -> COL0
- U1 pad 9: ROW0 -> COL1
Routing:
- net GND: track 840.5 -> 188.8 mm, vias 8 -> 0
- net +5V: track 757.3 -> 111.4 mm, vias 8 -> 5
- net COL6: track 395.5 -> 26.1 mm
- net COL8: track 375.1 -> 29.6 mm
- net COL7: track 371.7 -> 27.8 mm
- net COL13: track 376.7 -> 42.7 mm
- net COL12: track 370.2 -> 42.6 mm, vias 2 -> 0
- net COL10: track 341.8 -> 33.1 mm
- net COL9: track 338.4 -> 31.4 mm
- net COL11: track 348.0 -> 43.5 mm
- net COL5: track 303.7 -> 24.3 mm
- net ROW2: track 349.5 -> 86.2 mm, vias 8 -> 0
- net ROW1: track 335.4 -> 89.9 mm, vias 2 -> 0
- net ROW4: track 318.6 -> 81.7 mm, vias 2 -> 0
- net ROW0: track 325.7 -> 93.6 mm, vias 4 -> 0
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- added copper zone on F.Cu, net GND
- removed copper zone on B.Cu, net GND
Other:
- board size 285 x 95.1 mm -> 170 x 51.5 mm
- board text added: "150mm"
- board text added: "170mm"
- board text added: "Break off tab if original controller size is 150mm"
- board text added: "Ground pad for connection to backplate"
- board text added: "When installing sockets, compare the orientation to the stock controller"
- board text removed: "60-ALPS"
- board text removed: "PCB Revision 1.0"
- board text removed: "VOYAGER"
