File: ssk-controller.sch (KiCad schematic (older format))
At the start: 201 parts, among them SW1 5.2x5.2mm, U1 ATmega32U4-MU, U2 PRTR5V0U2X, Y1 16Mhz

Commit message: Finish board
Parts:
- removed C1, C10, C11, C12, C13, C14, C15, C16, C17, C18, C19, C20, C21, C9: 0.1uF, Capacitors_SMD:C_0603, symbol Device:C_Small
- removed D1, D10, D11, D12, D13, D14, D16, D17, D18, D19, D2, D20, D21, D22, D23, D24, D25, D26, D27, D28, D29, D3, D30, D31, D32, D33, D34, D35, D36, D37, D38, D39, D4, D40, D41, D42, D43, D44, D45, D46, D47, D48, D49, D5, D50, D51, D52, D53, D54, D55, D56, D57, D58, D59, D6, D60, D61, D62, D63, D64, D65, D67, D68, D7, D8, D9: SOD-123, Diodes_SMD:D_SOD-123, symbol Device:D_Small
- removed K_#1, K_#10, K_#2, K_#3, K_#4, K_#5, K_#6, K_#7, K_#8, K_#9, K_'1, K_,1, K_-1, K_.1, K_/1, K_;1, K_=1, K_A1, K_B1, K_C1, K_D1, K_E1, K_ENTER2, K_ENTER3, K_ENTER4, K_ESC1, K_ESC2, K_F1, K_G1, K_H1, K_I1, K_J1, K_K1, K_L1, K_M1, K_N1, K_O1, K_P1, K_Q1, K_R1, K_RWIN3, K_S1, K_SBACK1, K_SBACK2, K_SHIFT3, K_SRSHIFT2, K_T1, K_U1, K_V1, K_W1, K_WIN2, K_X1, K_Y1, K_Z1, K_[1, K_\2, K_]1: MX-1U, MX_Alps_Hybrid:ALPS-1U, symbol MX_Alps_Hybrids:MX-1U
- removed K_ALT1, K_CAPS2, K_CTRL1, K_RALT2, K_RCTRL2, K_RMENU2, K_RWIN1, K_RWIN2, K_SHIFT2, K_SPACE5, K_WIN1, K_WIN3: MX-1.25U, MX_Alps_Hybrid:ALPS-1.25U, symbol MX_Alps_Hybrids:MX-1U
- removed K_ALT2, K_ALT3, K_CAPS3, K_CTRL2, K_RALT1, K_RALT3, K_RCTRL3, K_TAB1, K_\1: MX-1.5U, MX_Alps_Hybrid:ALPS-1.5U, symbol MX_Alps_Hybrids:MX-1U
- removed K_BACK1: MX-2U, MX_Alps_Hybrid:ALPS-2U, symbol MX_Alps_Hybrids:MX-1U
- removed K_CAPS1, K_SRSHIFT1: MX-1.75U, MX_Alps_Hybrid:ALPS-1.75U, symbol MX_Alps_Hybrids:MX-1U
- removed K_ENTER1, K_SHIFT1, K_SPACE3: MX-2.25U, MX_Alps_Hybrid:ALPS-2.25U, symbol MX_Alps_Hybrids:MX-1U
- removed K_RSHIFT1, K_SPACE4: MX-2.75U, MX_Alps_Hybrid:ALPS-2.75U, symbol MX_Alps_Hybrids:MX-1U
- removed K_SPACE1: MX-7U, MX_Alps_Hybrid:ALPS-7U, symbol MX_Alps_Hybrids:MX-1U
- removed K_SPACE2: MX-6.25U, MX_Alps_Hybrid:ALPS-6.25U, symbol MX_Alps_Hybrids:MX-1U
- removed RGB1, RGB10, RGB11, RGB12, RGB13, RGB14, RGB2, RGB3, RGB4, RGB5, RGB6, RGB7, RGB8, RGB9: WS2812B, WS2812B:WS2812B, symbol ws2812b:WS2812B
- removed SW1: 5.2x5.2mm, Molex-0548190589:SKQG-1155865, symbol Voyager60-rescue:SW_Push
- removed U1: ATmega32U4-MU, Housings_DFN_QFN:QFN-44-1EP_7x7mm_Pitch0.5mm, symbol Voyager60-rescue:ATmega32U4-MU-MCU_Microchip_ATmega
- added J1: Conn_01x16, Pin_Headers:Pin_Header_Straight_1x16_Pitch2.54mm, symbol Connector_Generic:Conn_01x16
- added J2: Conn_01x08, Pin_Headers:Pin_Header_Straight_1x08_Pitch2.54mm, symbol Connector_Generic:Conn_01x08
- added J3: Conn_01x01, Pin_Headers:Pin_Header_Straight_1x01_Pitch2.54mm, symbol Connector_Generic:Conn_01x01
- added SW1: SW_Push, random-keyboard-parts:SKQG-1155865, symbol Switch:SW_Push
- added U1: ATmega32U4-AU, Housings_QFP:TQFP-44_10x10mm_Pitch0.8mm, symbol MCU_Microchip_ATmega:ATmega32U4-AU
- C2, C3, C4, C5, C6, C7, C8: footprint Capacitors_SMD:C_0603 -> Capacitors_SMD:C_0805
Connections:
- net labels added: COL14, COL15, ROW5, ROW6, ROW7
- net labels removed: RGBLED
- wire segments 646 -> 89
- no-connect marks 2 -> 1
Other:
- moved on the sheet: C2, C3, C4, C5, C6, C7, C8, R70, R71, Y1
