File: ssk-controller.sch (KiCad schematic (older format))
At the start: 22 parts, among them J1 Conn_01x16, J2 Conn_01x08, J3 Conn_01x01, SW1 SW_Push, U1 ATmega32U4-AU, U2 PRTR5V0U2X, Y1 16Mhz

Commit message: New gerbers for USB B
Parts:
- removed R73, R74: 5.1k, Resistors_SMD:R_0805, symbol Device:R_Small
- removed USB1: HRO-TYPE-C-31-M-12, Type-C:HRO-TYPE-C-31-M-12-Assembly, symbol Type-C:HRO-TYPE-C-31-M-12
- added J4: USB_B, locallib:TE-292304-2, symbol Connector:USB_B
Connections:
- wire segments 89 -> 64
Other:
- moved on the sheet: F1, R67, R68, U2
